Commit message: add simulation config and change moveit params

File: ur_description/urdf/inc/ur_macro.xacro (robot description, xacro)
@@ -64,5 +64,5 @@
     <xacro:ur_arm_transmission prefix="${prefix}" hw_interface="${transmission_hw_interface}" />
     <!-- links: main serial chain -->
-    <link name="${prefix}base_link"/>
+    <link name="${prefix}ur5e_base_link"/>
     <link name="${prefix}base_link_inertia">
       <visual>
@@ -207,6 +207,6 @@
     </link>
     <!-- joints: main serial chain -->
-    <joint name="${prefix}base_link-base_link_inertia" type="fixed">
-      <parent link="${prefix}base_link" />
+    <joint name="${prefix}ur5e_base_link-base_link_inertia" type="fixed">
+      <parent link="${prefix}ur5e_base_link" />
       <child link="${prefix}base_link_inertia" />
       <!-- 'base_link' is REP-103 aligned (so X+ forward), while the internal
@@ -291,5 +291,5 @@
     <!-- ROS-Industrial 'base' frame: base_link to UR 'Base' Coordinates transform -->
     <link name="${prefix}base"/>
-    <joint name="${prefix}base_link-base_fixed_joint" type="fixed">
+    <joint name="${prefix}ur5e_base_link-base_fixed_joint" type="fixed">
       <!-- Note the rotation over Z of pi radians: as base_link is REP-103
            aligned (ie: has X+ forward, Y+ left and Z+ up), this is needed
@@ -298,5 +298,5 @@
       -->
       <origin xyz="0 0 0" rpy="0 0 ${pi}"/>
-      <parent link="${prefix}base_link"/>
+      <parent link="${prefix}ur5e_base_link"/>
       <child link="${prefix}base"/>
     </joint>
